File: KiCAD-PCB/Amplificador2EtapasBJT.kicad_pcb (KiCad board)
At the start: 2 copper layers, 93 x 50.3 mm, 38 parts, among them J1 Vin, J2 CC, J3 Vout, Q1 NPN, Q2 NPN, Q3 NPN, Q4 NPN, Q5 PNP

Commit message: Correccion de Esquematico y PCB
Parts:
- RB3: value 180k -> 120k
- RB3-2: value 33k -> 27k
- RC1: value 10k -> 6.8k
- REQ4: value 22 -> 10
- moved Cc1 21.9 mm to (131.2, 105.8)
- moved REQ2 2.21 mm to (126.9, 101.7)
Connections:
- Cc1 pad 1: Net-(JP3-B) -> Net-(Q2-E)
- Q5 pad 1: Net-(Q4-C) -> Net-(Q4-E)
- Q5 pad 2: Net-(Q4-E) -> Net-(Q4-C)
Routing:
- net Net-(JP7-A): track 10.9 -> 33.7 mm
- net Net-(Q2-E): track 4.77 -> 16.8 mm
Changed lines of the file:
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@@
       (stroke (width 0.1) (type solid)) (layer "F.Fab"))
     (pad "1" thru_hole rect (at 0 0 90) (size 1.8 1.8) (drill 0.5) (layers "*.Cu" "*.Mask")
-      (net 22 "Net-(Q4-C)") (pinfunction "C") (pintype "open_collector"))
+      (net 7 "Net-(Q4-E)") (pinfunction "C") (pintype "open_collector"))
     (pad "2" thru_hole oval (at 2.54 0 90) (size 1.8 1.8) (drill 0.5) (layers "*.Cu" "*.Mask")
-      (net 7 "Net-(Q4-E)") (pinfunction "B") (pintype "input"))
+      (net 22 "Net-(Q4-C)") (pinfunction "B") (pintype "input"))
     (pad "3" thru_hole oval (at 5.08 0 90) (size 1.8 1.8) (drill 0.5) (layers "*.Cu" "*.Mask")
       (net 24 "Net-(JP10-B)") (pinfunction "E") (pintype "open_emitter"))
@@
   )
   (footprint "Capacitor_THT:CP_Radial_D6.3mm_P2.50mm" (layer "F.Cu")
-    (at 128.569 84.023)
+    (at 131.191 105.791)
     (descr "CP, Radial series, Radial, pin pitch=2.50mm, , diameter=6.3mm, Electrolytic Capacitor")
     (tags "CP Radial series Radial pin pitch 2.50mm  diameter 6.3mm Electrolytic Capacitor")
@@
       (stroke (width 0.1) (type solid)) (fill none) (layer "F.Fab"))
     (pad "1" thru_hole rect (at 0 0) (size 1.6 1.6) (drill 0.5) (layers "*.Cu" "*.Mask")
-      (net 2 "Net-(JP3-B)") (pintype "passive"))
+      (net 20 "Net-(Q2-E)") (pintype "passive"))
     (pad "2" thru_hole circle (at 2.5 0) (size 1.6 1.6) (drill 0.5) (layers "*.Cu" "*.Mask")
       (net 3 "Net-(JP7-A)") (pintype "passive"))
@@
         (effects (font (size 1 1) (thickness 0.15)))
     )
-    (fp_text value "22" (at 36.068 0 -90) (layer "F.Fab")
+    (fp_text value "10" (at 36.068 0 -90) (layer "F.Fab")
         (effects (font (size 1 1) (thickness 0.15)))
     )
@@
         (effects (font (size 1 1) (thickness 0.15)))
     )
-    (fp_text value "180k" (at 6.096 0 90) (layer "F.Fab")
+    (fp_text value "120k" (at 6.096 0 90) (layer "F.Fab")
         (effects (font (size 1 1) (thickness 0.15)))
     )
@@
   )
   (footprint "Resistor_THT:R_Axial_DIN0207_L6.3mm_D2.5mm_P10.16mm_Horizontal" (layer "F.Cu")
-    (at 129.037 101.295 -90)
+    (at 126.873 101.727 -90)
     (descr "Resistor, Axial_DIN0207 series, Axial, Horizontal, pin pitch=10.16mm, 0.25W = 1/4W, length*diameter=6.3*2.5mm^2, http://cdn-reichelt.de/documents/datenblatt/B400/1_4W%23YAG.pdf")
     (tags "Resistor Axial_DIN0207 series Axial Horizontal pin pitch 10.16mm 0.25W = 1/4W length 6.3mm diameter 2.5mm")
@@
         (effects (font (size 1 1) (thickness 0.15)))
     )
-    (fp_text value "33k" (at 6.604 0 90) (layer "F.Fab")
+    (fp_text value "27k" (at 6.604 0 90) (layer "F.Fab")
         (effects (font (size 1 1) (thickness 0.15)))
     )
@@
         (effects (font (size 1 1) (thickness 0.15)))
     )
-    (fp_text value "10k" (at 6.096 0 90) (layer "F.Fab")
+    (fp_text value "6.8k" (at 6.096 0 90) (layer "F.Fab")
         (effects (font (size 1 1) (thickness 0.15)))
     )
@@
   (segment (start 128.587 91.633) (end 128.587 84.041) (width 1) (layer "B.Cu") (net 2))
   (segment (start 127.513 73.863) (end 127.513 82.967) (width 1) (layer "B.Cu") (net 2))
+  (segment (start 133.691 86.645) (end 131.069 84.023) (width 1) (layer "B.Cu") (net 3))
   (segment (start 131.069 84.023) (end 131.069 75.636) (width 1) (layer "B.Cu") (net 3))
+  (segment (start 133.691 105.791) (end 133.691 86.645) (width 1) (layer "B.Cu") (net 3))
   (segment (start 131.069 75.636) (end 132.842 73.863) (width 1) (layer "B.Cu") (net 3))
   (segment (start 115.361 100.319) (end 108.717 93.675) (width 1) (layer "B.Cu") (net 5))
@@
   (segment (start 121.925 108.407) (end 121.417 107.899) (width 1) (layer "B.Cu") (net 19))
   (segment (start 121.417 107.899) (end 121.417 96.723) (width 1) (layer "B.Cu") (net 19))
-  (segment (start 129.037 101.295) (end 129.037 97.163) (width 1) (layer "B.Cu") (net 20))
-  (segment (start 129.037 97.163) (end 128.587 96.713) (width 1) (layer "B.Cu") (net 20))
+  (segment (start 126.873 98.425) (end 128.585 96.713) (width 1) (layer "B.Cu") (net 20))
+  (segment (start 126.873 101.727) (end 126.873 98.425) (width 1) (layer "B.Cu") (net 20))
+  (segment (start 128.585 96.713) (end 128.587 96.713) (width 1) (layer "B.Cu") (net 20))
+  (segment (start 130.114 96.713) (end 128.587 96.713) (width 1) (layer "B.Cu") (net 20))
+  (segment (start 131.191 105.791) (end 131.191 97.79) (width 1) (layer "B.Cu") (net 20))
+  (segment (start 131.191 97.79) (end 130.114 96.713) (width 1) (layer "B.Cu") (net 20))
   (segment (start 145.293 103.327) (end 147.325 105.359) (width 1) (layer "B.Cu") (net 21))
   (segment (start 147.325 105.359) (end 153.929 105.359) (width 1) (layer "B.Cu") (net 21))
@@
     (polygon
       (pts
-        (xy 100.081 66.751)
-        (xy 193.553 66.751)
-        (xy 193.553 117.043)
-        (xy 100.081 117.043)
+        (xy 193.294 117.094)
+        (xy 193.294 66.675)
+        (xy 100.33 66.675)
+        (xy 100.33 117.221)
       )
     )

Commit message: Actualizacion del Sch y PCB a corregir
Parts:
- removed Cc1: 10uF, Capacitor_THT:CP_Radial_D6.3mm_P2.50mm
- removed TP3: TPBQ5, Connector_PinHeader_2.54mm:PinHeader_1x01_P2.54mm_Vertical
- added Ci2: 1000uF, Capacitor_THT:CP_Radial_D10.0mm_P5.00mm, F.Cu at (119.2, 92.8)
- added Co3: 10uF, Capacitor_THT:CP_Radial_D6.3mm_P2.50mm, F.Cu at (186.3, 73.3)
- added RBQ4: 100, Resistor_THT:R_Axial_DIN0207_L6.3mm_D2.5mm_P10.16mm_Horizontal, F.Cu at (177.0, 103.0)
- added Rout2: 15, Resistor_THT:R_Axial_DIN0207_L6.3mm_D2.5mm_P10.16mm_Horizontal, F.Cu at (183.8, 94.4)
- added TP4: TPB-Q2, Connector_PinHeader_2.54mm:PinHeader_1x01_P2.54mm_Vertical, F.Cu at (123.4, 109.4)
- Co2: footprint Capacitor_THT:CP_Radial_D6.3mm_P2.50mm -> Capacitor_THT:CP_Radial_Tantal_D6.0mm_P5.00mm
- Q1, Q3: footprint Package_TO_SOT_THT:TO-92L_Inline_Wide -> Package_TO_SOT_THT:TO-92_Inline_Wide
- Q2: footprint Package_TO_SOT_THT:TO-92L_Inline_Wide -> Package_TO_SOT_THT:TO-126-3_Vertical
- Q4: footprint Package_TO_SOT_THT:TO-92L_Inline_Wide -> Package_TO_SOT_THT:TO-220-3_Vertical
- Q5: footprint Package_TO_SOT_THT:TO-126-3_Vertical -> Package_TO_SOT_THT:TO-220-3_Vertical
- REQ2: value 470 -> 47
- Rout1: value 7.5 -> 15; footprint Resistor_THT:R_Axial_DIN0414_L11.9mm_D4.5mm_P15.24mm_Horizontal -> Resistor_THT:R_Axial_DIN0207_L6.3mm_D2.5mm_P10.16mm_Horizontal
- moved Co1 51.6 mm to (138.6, 108.8)
- moved Q2 14.8 mm to (141.8, 84.9), turned to 180 degrees
- moved RB3 12.9 mm to (150.5, 84.3)
- moved Q4 12.7 mm to (166.7, 104.2), turned to 90 degrees
- moved Rbin1 12.2 mm to (127.1, 79.4)
- moved TP1 12.0 mm to (117.0, 111.7)
- moved Rout1 11.4 mm to (186.3, 94.4)
- moved Q5 11.0 mm to (175.5, 89.2), turned to 180 degrees
- moved Q3 10.3 mm to (155.5, 92.2)
- moved Co2 9.61 mm to (156.5, 103.0)
- moved J1 9.40 mm to (112.1, 106.1)
- moved RB3-2 9.36 mm to (146.9, 102.7)
- moved J2 8.62 mm to (112.5, 81.4)
- moved RL1 8.43 mm to (190.2, 90.0)
- moved Ci1 8.27 mm to (123.6, 102.1)
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Connections:
- Co1 pad 1: Net-(Co1-Pad1) -> Net-(Q2-E)
- Co1 pad 2: Net-(JP9-A) -> Net-(JP7-A)
- J3 pad 1: Net-(J3-Pin_1) -> Earth
- J3 pad 2: Earth -> Net-(J3-Pin_2)
- JP9 pad 2: Net-(J3-Pin_1) -> Net-(J3-Pin_2)
- Q2 pad 1: Net-(JP3-B) -> Net-(Q1-E)
- Q2 pad 2: Net-(Q1-E) -> Net-(JP3-B)
- Q4 pad 1: Net-(Q4-C) -> Net-(Q4-B)
- Q4 pad 2: Net-(Q4-B) -> Net-(JP11-A)
- Q5 pad 2: Net-(Q4-C) -> Net-(JP11-B)
- RL1 pad 1: Net-(J3-Pin_1) -> Net-(J3-Pin_2)
- Rout1 pad 2: Net-(Co1-Pad1) -> Net-(Co3-Pad2)
Routing:
- net Earth: track 0.00 -> 96.3 mm
- net Net-(J3-Pin_1): track 74.6 -> 0.00 mm
- net Net-(J3-Pin_2): track 0.00 -> 74.5 mm
- net Net-(Q2-E): track 16.8 -> 43.9 mm
- net Net-(Q1-E): track 20.2 -> 37.9 mm
- net Net-(J2-Pin_2): track 86.4 -> 102.7 mm
- net Net-(JP11-B): track 0.00 -> 15.5 mm
- net Net-(JP11-A): track 0.00 -> 14.0 mm
- net Net-(Co3-Pad2): track 0.00 -> 13.5 mm
- net Net-(Q4-C): track 12.4 -> 0.00 mm
- net Net-(Co1-Pad1): track 9.29 -> 0.00 mm
- net Net-(JP8-B): track 27.6 -> 36.6 mm
- net Net-(Q4-E): track 63.6 -> 72.3 mm
- net Net-(Q4-B): track 29.3 -> 21.0 mm
- net Net-(JP7-A): track 33.7 -> 40.0 mm
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
Commit message: Imagenes del Setup de Proteus
Parts:
- Ci2: value 1000uF -> 10uF
- Co3: value 10uF -> 1000uF
- Q1: value NPN -> BC546 B NPN
- Q2: value NPN -> BD 139NPN
- moved Co2 5.25 mm to (161.8, 103.0), turned to 180 degrees
- moved Co3 2.52 mm to (183.8, 73.3), turned to 0 degrees
Connections:
- Co2 pad 1: Net-(JP8-B) -> Net-(Q4-B)
- Co2 pad 2: Net-(Q4-B) -> Net-(JP8-B)
- Co3 pad 1: Net-(JP9-A) -> Net-(Co3-Pad1)
- Co3 pad 2: Net-(Co3-Pad2) -> Net-(JP9-A)
- J1 pad 1: Earth -> Net-(J1-Pin_2)
- J1 pad 2: Net-(J1-Pin_2) -> Earth
- Q2 pad 1: Net-(Q1-E) -> Net-(JP3-B)
- Q2 pad 2: Net-(JP3-B) -> Net-(Q1-E)
- Q5 pad 1: Net-(Q4-E) -> Net-(Q5-B)
- Q5 pad 2: Net-(JP11-B) -> Net-(Q4-E)
- RBQ4 pad 1: Net-(JP11-B) -> Net-(Q5-B)
- Rout1 pad 2: Net-(Co3-Pad2) -> Net-(Co3-Pad1)
- Rout2 pad 2: Net-(Co3-Pad2) -> Net-(Co3-Pad1)
Routing:
- net Net-(JP11-B): track 15.5 -> 0.00 mm
- net Net-(Q5-B): track 0.00 -> 14.5 mm
- net Net-(Co3-Pad2): track 13.5 -> 0.00 mm
- net Net-(Co3-Pad1): track 0.00 -> 13.5 mm
- net Net-(Q4-E): track 72.3 -> 60.5 mm
- net Net-(Q4-C): track 14.0 -> 19.6 mm
- net Net-(JP8-B): track 36.6 -> 36.0 mm

Commit message: pusheo un monotn de cosas
Parts:
- Rout1: value 15 -> 10
Connections:
- J1 pad 1: Net-(J1-Pin_2) -> Earth
- J1 pad 2: Earth -> Net-(J1-Pin_2)
- Q3 pad 1: Net-(JP8-A) -> Net-(Q3-C)
- Q4 pad 1: Net-(Q4-B) -> Net-(Q4-C)
- Q4 pad 2: Net-(Q4-C) -> Net-(JP8-B)
- Q5 pad 1: Net-(Q5-B) -> Net-(Q4-E)
- Q5 pad 2: Net-(Q4-E) -> Net-(Q5-B)
- R1Q4 pad 1: Net-(Q4-B) -> Net-(JP8-B)
- R2Q4 pad 2: Net-(Q4-B) -> Net-(JP8-B)
- RC1 pad 2: Net-(JP8-A) -> Net-(Q3-C)
Routing:
- net Net-(Q4-B): track 20.7 -> 0.00 mm
- net (no net): track 0.00 -> 20.7 mm
